File: Connectors.kicad_sch (KiCad schematic)
At the start: 4 parts, among them J7 DS1013-20SSIB1-B-0

Commit message: Поменял десат подключение, сделал зазоры на силовых полигонах
Parts:
- Q2: value ~ -> (none)
