File: Driver_1.kicad_sch (KiCad schematic)
At the start: 43 parts, among them Q1 C3M0065100K, Q3 C3M0065100K

Commit message: Поменял десат подключение, сделал зазоры на силовых полигонах
Parts:
- C90, C91, D31, D32, D33, D34, D35, D36, D4, D58, D59, D6, J1, J2, J3: value ~ -> (none)
Connections:
- net DS1 is gone; now on net D2: C61.2, C90.1, D32.3 (GND2), D33.2 (A), Q1.3 (DS), R104.1, R2.1
- net D1: now also D4.1 (K)
- net D2: now also D6.1 (K); no longer D4.1 (K)
- net DS2: now also C25.2, C26.2, J2.1 (Pin_1), Q3.2 (S)
- removed net S2: C25.2, C26.2, D6.1 (K), J2.1 (Pin_1), Q3.2 (S)
